Commit message: feat: phase 1 complete - teleop via ros2_control + ESP32-C6 serial

File: src/plaguebot_base_description/urdf/plaguebot_base.urdf.xacro (robot description, xacro)
@@ -1,4 +1,5 @@
 <?xml version="1.0"?>
 <robot xmlns:xacro="http://www.ros.org/wiki/xacro" name="plaguebot_base">
+  <xacro:arg name="is_sim" default="true"/>
   <!-- PROPIEDADES FÍSICAS — No modificar sin consultar -->
   <xacro:property name="wheel_radius"    value="0.0762"/>
@@ -16,4 +17,5 @@
     <color rgba="0.18 0.18 0.18 1.0"/>
   </material>
+  <xacro:if value="$(arg is_sim)">
   <gazebo>
     <plugin filename="gz_ros2_control-system" name="gz_ros2_control::GazeboSimROS2ControlPlugin">
@@ -21,5 +23,7 @@
     </plugin>
   </gazebo>
+  </xacro:if>
   <xacro:include filename="$(find plaguebot_base_description)/urdf/plaguebot_base_ros2_control.xacro"/>
+  <xacro:plaguebot_ros2_control is_sim="$(arg is_sim)"/>
   <!-- BASE FOOTPRINT (raíz del robot, proyección al suelo) -->
   <link name="base_footprint"/>

File: src/plaguebot_base_description/urdf/plaguebot_base_ros2_control.xacro (robot description, xacro)
@@ -1,28 +1,56 @@
 <?xml version="1.0"?>
 <robot xmlns:xacro="http://www.ros.org/wiki/xacro">
-  <ros2_control name="plaguebot_base" type="system">
-    <hardware>
-      <plugin>gz_ros2_control/GazeboSimSystem</plugin>
-    </hardware>
-    <joint name="front_left_wheel_joint">
-      <command_interface name="velocity"/>
-      <state_interface name="position"/>
-      <state_interface name="velocity"/>
-    </joint>
-    <joint name="front_right_wheel_joint">
-      <command_interface name="velocity"/>
-      <state_interface name="position"/>
-      <state_interface name="velocity"/>
-    </joint>
-    <joint name="rear_left_wheel_joint">
-      <command_interface name="velocity"/>
-      <state_interface name="position"/>
-      <state_interface name="velocity"/>
-    </joint>
-    <joint name="rear_right_wheel_joint">
-      <command_interface name="velocity"/>
-      <state_interface name="position"/>
-      <state_interface name="velocity"/>
-    </joint>
-  </ros2_control>
+  <xacro:macro name="plaguebot_ros2_control" params="is_sim:=true">
+    <ros2_control name="plaguebot_base" type="system">
+      <!-- Simulation -->
+      <xacro:if value="${is_sim}">
+        <hardware>
+          <plugin>gz_ros2_control/GazeboSimSystem</plugin>
+        </hardware>
+        <joint name="front_left_wheel_joint">
+          <command_interface name="velocity"/>
+          <state_interface name="position"/>
+          <state_interface name="velocity"/>
+        </joint>
+        <joint name="front_right_wheel_joint">
+          <command_interface name="velocity"/>
+          <state_interface name="position"/>
+          <state_interface name="velocity"/>
+        </joint>
+        <joint name="rear_left_wheel_joint">
+          <command_interface name="velocity"/>
+          <state_interface name="position"/>
+          <state_interface name="velocity"/>
+        </joint>
+        <joint name="rear_right_wheel_joint">
+          <command_interface name="velocity"/>
+          <state_interface name="position"/>
+          <state_interface name="velocity"/>
+        </joint>
+      </xacro:if>
+      <!-- Real Robot -->
+      <xacro:unless value="${is_sim}">
+        <hardware>
+          <plugin>plaguebot_firmware/PlaguebotInterface</plugin>
+          <param name="port">/dev/ttyACM0</param>
+        </hardware>
+        <joint name="front_right_wheel_joint">
+          <command_interface name="velocity">
+            <param name="min">-7</param>
+            <param name="max">7</param>
+          </command_interface>
+          <state_interface name="position"/>
+          <state_interface name="velocity"/>
+        </joint>
+        <joint name="front_left_wheel_joint">
+          <command_interface name="velocity">
+            <param name="min">-7</param>
+            <param name="max">7</param>
+          </command_interface>
+          <state_interface name="position"/>
+          <state_interface name="velocity"/>
+        </joint>
+      </xacro:unless>
+    </ros2_control>
+  </xacro:macro>
 </robot>
