Commit message: chore(phase2): wrap up base+arm integration leftovers
Pre-existing Phase 2 changes that close out the unified robot integration:
- plaguebot.urdf.xacro: add is_standalone arg (default true) gating the
  world link + virtual_joint, so the arm can be embedded in the unified
  plaguebot_robot URDF without a second world root (ADR 0001). Mesh
  collisions are untouched.
- plaguebot_gazebo.xacro: gate the arm-only controller_manager behind
  is_standalone; the unified URDF provides one combined manager.
- base_controllers.yaml: document the intentional wheel-naming inversion
  (ADR 0002) so the swapped left/right wheel lists aren't read as a bug.
- plaguebot.srdf: add 'folded' (compact stow for navigation) and 'deploy'
  (D435 angled at the plant row for scanning) arm group states.
- Track CLAUDE.md (project agent instructions).

Co-Authored-By: Claude Opus 4.8 <noreply@anthropic.com>

File: src/plaguebot_description/urdf/plaguebot.urdf.xacro (robot description, xacro)
@@ -2,4 +2,7 @@
 <robot xmlns:xacro="http://www.ros.org/wiki/xacro" name="plaguebot">
     <xacro:arg name="is_ignition" default="true"/>
+    <!-- When false, omits the world root link so the arm can be included in a
+         unified robot URDF (plaguebot_robot). See docs/adr/0001. -->
+    <xacro:arg name="is_standalone" default="true"/>
     <xacro:include filename="$(find plaguebot_description)/urdf/plaguebot_gazebo.xacro"/>
     <xacro:include filename="$(find plaguebot_description)/urdf/plaguebot_ros2_control.xacro"/>
@@ -16,5 +19,12 @@
         </inertial>
     </xacro:macro>
-    <link name="world"/>
+    <xacro:if value="$(arg is_standalone)">
+      <link name="world"/>
+      <joint name="virtual_joint" type="fixed">
+        <parent link="world"/>
+        <child link="base_link"/>
+        <origin rpy="0 0 0" xyz="0 0 0"/>
+      </joint>
+    </xacro:if>
     <link name="base_link">
         <xacro:default_inertial mass="1.0"/>
@@ -35,9 +45,4 @@
         </collision>
     </link>
-    <joint name="virtual_joint" type="fixed">
-        <parent link="world"/>
-        <child link="base_link"/>
-        <origin rpy="0 0 0" xyz="0 0 0"/>
-    </joint>
     <link name="base_plate_link">
         <xacro:default_inertial mass="0.1"/>

File: src/plaguebot_description/urdf/plaguebot_gazebo.xacro (robot description, xacro)
@@ -1,5 +1,9 @@
 <?xml version="1.0"?>
 <robot xmlns:xacro="http://www.ros.org/wiki/xacro" name="plaguebot">
-    <gazebo>
+    <!-- Arm-only controller_manager — only when running the arm standalone.
+         When is_standalone=false the unified plaguebot_robot URDF provides
+         a single combined controller_manager for base + arm. -->
+    <xacro:if value="$(arg is_standalone)">
+      <gazebo>
         <xacro:if value="$(arg is_ignition)">
             <plugin filename="ign_ros2_control-system" name="ign_ros2_control::IgnitionROS2ControlPlugin">
@@ -12,4 +16,5 @@
             </plugin>
         </xacro:unless>
-    </gazebo>
+      </gazebo>
+    </xacro:if>
 </robot>
