Commit message: Base bringup on real robot: ESP32 bridge, calibrated motor/encoder mapping, EKF for real sensors
- esp32_bridge: serial <-> ROS 2 bridge (odom + IMU out, cmd_vel/arm in)
  with per-motor sign; M4 (rear-right) wired reversed -> motor_signs=[1,1,1,-1]
- calibrate_base: standalone pulse/watch/verify helper for encoder + motor
  mapping; verify drives each wheel forward through the bridge's sign logic
- ekf: fuse real /odom vx and IMU yaw-rate only (real IMU has no absolute
  orientation); use_sim_time=false
- urdf/launch: real-robot base bringup

Encoder->wheel: E1=front-left, E2=front-right, E3=rear-left, E4=rear-right (all +)
Motor->wheel:   M1..M4 = same corners; M4 forward channel inverted in software

Co-Authored-By: Claude Opus 4.7 <noreply@anthropic.com>

File: src/plaguebot_bringup/urdf/plaguebot_base.urdf.xacro (robot description, xacro)
@@ -1,7 +1,5 @@
 <?xml version="1.0"?>
 <robot xmlns:xacro="http://www.ros.org/wiki/xacro" name="plaguebot_base">
-  <xacro:arg name="is_sim" default="true"/>
-  <!-- Override in unified robot to use a combined YAML (base + arm controllers) -->
-  <xacro:arg name="controllers_yaml" default="$(find plaguebot_base_description)/config/base_controllers.yaml"/>
+  <xacro:arg name="is_sim" default="false"/>
   <!-- PROPIEDADES FÍSICAS — No modificar sin consultar -->
   <xacro:property name="wheel_radius"    value="0.0762"/>
@@ -26,6 +24,6 @@
   </gazebo>
   </xacro:if>
-  <xacro:include filename="$(find plaguebot_base_description)/urdf/plaguebot_base_ros2_control.xacro"/>
-  <xacro:plaguebot_ros2_control is_sim="$(arg is_sim)"/>
+  <!-- Real robot: motion is owned by esp32_bridge (not ros2_control), so the
+       ros2_control block is intentionally omitted here. -->
   <!-- BASE FOOTPRINT (raíz del robot, proyección al suelo) -->
   <link name="base_footprint"/>
@@ -40,5 +38,5 @@
       <origin xyz="-0.30 0.41 -0.04" rpy="1.5708 0.0 0.0"/>
         <geometry>
-          <mesh filename="package://plaguebot_base_description/meshes/visual/CHASIS_PLAGUEBOT.STL" scale="0.001 0.001 0.001"/>
+          <mesh filename="package://plaguebot_bringup/meshes/visual/CHASIS_PLAGUEBOT.STL" scale="0.001 0.001 0.001"/>
         </geometry>
         <material name="aluminum"/>
@@ -47,5 +45,5 @@
        <origin xyz="-0.30 0.41 -0.04" rpy="1.5708 0.0 0.0"/>
         <geometry>
-          <mesh filename="package://plaguebot_base_description/meshes/visual/CHASIS_PLAGUEBOT.STL" scale="0.001 0.001 0.001"/>
+          <mesh filename="package://plaguebot_bringup/meshes/visual/CHASIS_PLAGUEBOT.STL" scale="0.001 0.001 0.001"/>
         </geometry>
     </collision>
@@ -87,5 +85,5 @@
       <origin xyz="0.027 -0.0348 0" rpy="1.5708 0 -3.1416"/>
       <geometry>
-        <mesh filename="package://plaguebot_base_description/meshes/visual/RPLIDAR_C1.STL" scale="0.001 0.001 0.001"/>
+        <mesh filename="package://plaguebot_bringup/meshes/visual/RPLIDAR_C1.STL" scale="0.001 0.001 0.001"/>
       </geometry>
       <material name="lidar_black"/>
@@ -115,5 +113,5 @@
       <origin xyz="-0.15 0.16 0.04" rpy="-1.5708 0.0 0.0"/>
         <geometry>
-          <mesh filename="package://plaguebot_base_description/meshes/visual/LLANTA.STL" scale="0.001 0.001 0.001"/>
+          <mesh filename="package://plaguebot_bringup/meshes/visual/LLANTA.STL" scale="0.001 0.001 0.001"/>
         </geometry>
         <material name="tire_black"/>
@@ -122,5 +120,5 @@
        <origin xyz="-0.15 0.16 0.04" rpy="-1.5708 0.0 0.0"/>
         <geometry>
-          <mesh filename="package://plaguebot_base_description/meshes/visual/LLANTA.STL" scale="0.001 0.001 0.001"/>
+          <mesh filename="package://plaguebot_bringup/meshes/visual/LLANTA.STL" scale="0.001 0.001 0.001"/>
         </geometry>
     </collision>
@@ -141,5 +139,5 @@
       <origin xyz="-0.15 0.16 0.04" rpy="-1.5708 0.0 0.0"/>
         <geometry>
-          <mesh filename="package://plaguebot_base_description/meshes/visual/LLANTA.STL" scale="0.001 0.001 0.001"/>
+          <mesh filename="package://plaguebot_bringup/meshes/visual/LLANTA.STL" scale="0.001 0.001 0.001"/>
         </geometry>
         <material name="tire_black"/>
@@ -148,5 +146,5 @@
        <origin xyz="-0.15 0.16 0.04" rpy="-1.5708 0.0 0.0"/>
         <geometry>
-          <mesh filename="package://plaguebot_base_description/meshes/visual/LLANTA.STL" scale="0.001 0.001 0.001"/>
+          <mesh filename="package://plaguebot_bringup/meshes/visual/LLANTA.STL" scale="0.001 0.001 0.001"/>
         </geometry>
     </collision>
@@ -167,5 +165,5 @@
       <origin xyz="-0.15 -0.16 -0.04" rpy="1.5708 0.0 0.0"/>
         <geometry>
-          <mesh filename="package://plaguebot_base_description/meshes/visual/LLANTA.STL" scale="0.001 0.001 0.001"/>
+          <mesh filename="package://plaguebot_bringup/meshes/visual/LLANTA.STL" scale="0.001 0.001 0.001"/>
         </geometry>
         <material name="tire_black"/>
@@ -174,5 +172,5 @@
        <origin xyz="-0.15 -0.16 -0.04" rpy="1.5708 0.0 0.0"/>
         <geometry>
-          <mesh filename="package://plaguebot_base_description/meshes/visual/LLANTA.STL" scale="0.001 0.001 0.001"/>
+          <mesh filename="package://plaguebot_bringup/meshes/visual/LLANTA.STL" scale="0.001 0.001 0.001"/>
         </geometry>
     </collision>
@@ -193,5 +191,5 @@
       <origin xyz="-0.15 -0.16 -0.04" rpy="1.5708 0.0 0.0"/>
         <geometry>
-          <mesh filename="package://plaguebot_base_description/meshes/visual/LLANTA.STL" scale="0.001 0.001 0.001"/>
+          <mesh filename="package://plaguebot_bringup/meshes/visual/LLANTA.STL" scale="0.001 0.001 0.001"/>
         </geometry>
         <material name="tire_black"/>
@@ -200,5 +198,5 @@
        <origin xyz="-0.15 -0.16 -0.04" rpy="1.5708 0.0 0.0"/>
         <geometry>
-          <mesh filename="package://plaguebot_base_description/meshes/visual/LLANTA.STL" scale="0.001 0.001 0.001"/>
+          <mesh filename="package://plaguebot_bringup/meshes/visual/LLANTA.STL" scale="0.001 0.001 0.001"/>
         </geometry>
     </collision>
